Commit message: 更新XBOX遥操作与数据采集代码

File: el_a3_ros/el_a3_description/urdf/el_a3.urdf (robot description, URDF)
Before this commit: robot EL-A3, 10 links, 9 joints
Joints:
- joint L7_joint: limit lower=-1.5708 upper=1.5708 effort=6.0 velocity=50 -> lower=-1.5708 upper=2.0 effort=6.0 velocity=50

File: el_a3_ros/el_a3_description/urdf/el_a3.urdf.xacro (robot description, xacro)
@@ -265,5 +265,5 @@
     <child link="gripper_link"/>
     <axis xyz="0 0 1"/>
-    <limit effort="${wrist_effort}" velocity="50" lower="-1.5708" upper="1.5708"/>
+    <limit effort="${wrist_effort}" velocity="50" lower="-1.5708" upper="2.0"/>
     <dynamics damping="0.05" friction="0.05"/>
   </joint>

File: el_a3_ros/el_a3_description/urdf/el_a3_ros2_control.xacro (robot description, xacro)
@@ -36,4 +36,8 @@
           <param name="kd_velocity_ref">1.0</param>        <!-- Reference velocity where Kd drops to midpoint (rad/s) -->
           <param name="kd_smoothing_alpha">0.15</param>    <!-- EMA smoothing factor (smaller = smoother transitions) -->
+          <!-- Gripper torque-limit hold (matches SDK/PICO GripperCtrl(gripper_effort=...)) -->
+          <param name="gripper_default_torque_limit">0.65</param>
+          <param name="gripper_torque_limit_epsilon">0.01</param>
+          <param name="gripper_hold_torque_ff">0.0</param>
           <!-- Pinocchio dynamics model configuration -->
           <param name="urdf_path">$(find el_a3_description)/urdf/el_a3.urdf</param>
@@ -233,5 +237,5 @@
         <command_interface name="position">
           <param name="min">-1.5708</param>
-          <param name="max">1.5708</param>
+          <param name="max">2.0</param>
         </command_interface>
         <command_interface name="velocity">
